Commit message: in progress add robot chasis and wheels

File: catkin_ws/src/my_robot/urdf/my_robot.xacro (robot description, xacro)
@@ -55,3 +55,56 @@
     </visual>
   </link>
+      <link name="left_wheel">
+        <pose>0.0 0.0 0.0 0 1.5707 1.5707</pose>
+        <collision name="collision">
+          <geometry>
+            <cylinder>
+              <radius>.1</radius>
+              <length>.05</length>
+            </cylinder>
+          </geometry>
+        </collision>
+        <visual name="visual">
+          <geometry>
+            <cylinder>
+              <radius>.1</radius>
+              <length>.05</length>
+            </cylinder>
+          </geometry>
+        </visual>
+    <mass value="5"/>
+      <inertia
+          ixx="0.1" ixy="0" ixz="0"
+          iyy="0.1" iyz="0"
+          izz="0.1"
+      />
+      </link>
+  <link name='right_wheel'>
+    <geometry>
+      <cylinder radius='0.1' length='0.05'/>
+    </geometry>
+    <origin xyz="0 0 0" rpy="0 1.5707 1.5707"/>
+    <mass value="5"/>
+      <inertia
+          ixx="0.1" ixy="0" ixz="0"
+          iyy="0.1" iyz="0"
+          izz="0.1"
+      />
+  </link>
+  <joint type="continuous" name="left_wheel_hinge">
+    <origin xyz="0 0.15 0" rpy="0 0 0"/>
+    <child link="left_wheel"/>
+    <parent link="chassis"/>
+    <axis xyz="0 1 0" rpy="0 0 0"/>
+    <limit effort="10000" velocity="1000"/>
+    <dynamics damping="1.0" friction="1.0"/>
+  </joint>
+  <joint type="continuous" name="right_wheel_hinge">
+    <origin xyz="0 -0.15 0" rpy="0 0 0"/>
+    <child link="right_wheel"/>
+    <parent link="chassis"/>
+    <axis xyz="0 1 0" rpy="0 0 0"/>
+    <limit effort="10000" velocity="1000"/>
+    <dynamics damping="1.0" friction="1.0"/>
+  </joint>
 </robot>

Commit message: configure robot wheels and joints

File: catkin_ws/src/my_robot/urdf/my_robot.xacro (robot description, xacro)
@@ -56,40 +56,48 @@
   </link>
       <link name="left_wheel">
-        <pose>0.0 0.0 0.0 0 1.5707 1.5707</pose>
         <collision name="collision">
+        <origin xyz="0.0 0 0" rpy=" 0 1.5707 1.5707"/>
           <geometry>
-            <cylinder>
-              <radius>.1</radius>
-              <length>.05</length>
-            </cylinder>
+            <cylinder radius="0.1" length="0.05"/>
           </geometry>
         </collision>
         <visual name="visual">
+        <origin xyz="0.0 0 0" rpy=" 0 1.5707 1.5707"/>
           <geometry>
-            <cylinder>
-              <radius>.1</radius>
-              <length>.05</length>
-            </cylinder>
+            <cylinder radius="0.1" length="0.05"/>
           </geometry>
         </visual>
-    <mass value="5"/>
-      <inertia
+       <inertial>
+        <mass value="5.0"/>
+        <inertia
           ixx="0.1" ixy="0" ixz="0"
           iyy="0.1" iyz="0"
           izz="0.1"
-      />
-      </link>
-  <link name='right_wheel'>
-    <geometry>
-      <cylinder radius='0.1' length='0.05'/>
-    </geometry>
-    <origin xyz="0 0 0" rpy="0 1.5707 1.5707"/>
-    <mass value="5"/>
-      <inertia
+        />
+      </inertial>
+    </link>
+      <link name="right_wheel">
+        <collision name="collision">
+        <origin xyz="0.0 0 0" rpy=" 0 1.5707 1.5707"/>
+          <geometry>
+            <cylinder radius="0.1" length="0.05"/>
+          </geometry>
+        </collision>
+        <visual name="visual">
+        <origin xyz="0.0 0 0" rpy=" 0 1.5707 1.5707"/>
+          <geometry>
+            <cylinder radius="0.1" length="0.05"/>
+          </geometry>
+        </visual>
+       <inertial>
+        <mass value="5.0"/>
+        <origin xyz="0.0 0 0" rpy=" 0 1.5707 1.5707"/>
+        <inertia
           ixx="0.1" ixy="0" ixz="0"
           iyy="0.1" iyz="0"
           izz="0.1"
-      />
-  </link>
+        />
+      </inertial>
+    </link>
   <joint type="continuous" name="left_wheel_hinge">
     <origin xyz="0 0.15 0" rpy="0 0 0"/>

Commit message: add camera

File: catkin_ws/src/my_robot/urdf/my_robot.xacro (robot description, xacro)
@@ -116,3 +116,31 @@
     <dynamics damping="1.0" friction="1.0"/>
   </joint>
+   <link name="camera">
+        <collision name="collision">
+         <origin xyz="0.0 0 0" rpy=" 0 0 0"/>
+          <geometry>
+            <box size="0.05 0.05 0.05"/>
+          </geometry>
+        </collision>
+        <visual name="visual">
+         <origin xyz="0.0 0 0" rpy=" 0 0 0"/>
+          <geometry>
+            <box size="0.05 0.05 0.05"/>
+          </geometry>
+        </visual>
+       <inertial>
+        <mass value="0.1"/>
+        <inertia
+          ixx="0.000001" ixy="0" ixz="0"
+          iyy="0.000001" iyz="0"
+          izz="0.000001"
+        />
+      </inertial>
+    </link>
+  <joint type="fixed" name="camera_joint">
+    <origin xyz="0.2 0 0" rpy="0 0 0"/>
+    <child link="camera"/>
+    <parent link="chassis"/>
+    <axis xyz="0 1 0" rpy="0 0 0"/>
+  </joint>
 </robot>

Commit message: add hokuyo laser and mesh

File: catkin_ws/src/my_robot/urdf/my_robot.xacro (robot description, xacro)
@@ -144,3 +144,31 @@
     <axis xyz="0 1 0" rpy="0 0 0"/>
   </joint>
+   <link name="hokuyo">
+        <collision name="collision">
+         <origin xyz="0.0 0 0" rpy=" 0 0 0"/>
+          <geometry>
+            <box size="0.1 0.1 0.1"/>
+          </geometry>
+        </collision>
+        <visual name="visual">
+         <origin xyz="0.0 0 0" rpy=" 0 0 0"/>
+          <geometry>
+            <mesh filename="package://my_robot/meshes/hokuyo.dae"/>
+          </geometry>
+        </visual>
+       <inertial>
+        <mass value="0.00001"/>
+        <inertia
+          ixx="0.000001" ixy="0" ixz="0"
+          iyy="0.000001" iyz="0"
+          izz="0.000001"
+        />
+      </inertial>
+    </link>
+  <joint type="fixed" name="hokuyo_joint">
+    <origin xyz="0.15 0.0 0.075" rpy="0 0 0"/>
+    <child link="hokuyo"/>
+    <parent link="chassis"/>
+    <axis xyz="0 1 0" rpy="0 0 0"/>
+  </joint>
 </robot>

Commit message: add plugins for camera, wheels and lidar and set up RViz

File: catkin_ws/src/my_robot/urdf/my_robot.xacro (robot description, xacro)
@@ -1,4 +1,5 @@
 <?xml version='1.0'?>
 <robot name="my_robot" xmlns:xacro="http://www.ros.org/wiki/xacro">
+  <xacro:include filename="$(find my_robot)/urdf/my_robot.gazebo" />
   <link name="robot_footprint"></link>
   <joint name="robot_footprint_joint" type="fixed">
@@ -172,3 +173,15 @@
     <axis xyz="0 1 0" rpy="0 0 0"/>
   </joint>
+<gazebo reference="chassis">
+    <material>Gazebo/Blue</material>
+</gazebo>
+<gazebo reference="left_wheel">
+    <material>Gazebo/Yellow</material>
+</gazebo>
+<gazebo reference="right_wheel">
+    <material>Gazebo/Yellow</material>
+</gazebo>
+<gazebo reference="camera">
+    <material>Gazebo/Orange</material>
+</gazebo>
 </robot>

Commit message: minor cleanup

File: catkin_ws/src/my_robot/urdf/my_robot.xacro (robot description, xacro)
@@ -176,12 +176,3 @@
     <material>Gazebo/Blue</material>
 </gazebo>
-<gazebo reference="left_wheel">
-    <material>Gazebo/Yellow</material>
-</gazebo>
-<gazebo reference="right_wheel">
-    <material>Gazebo/Yellow</material>
-</gazebo>
-<gazebo reference="camera">
-    <material>Gazebo/Orange</material>
-</gazebo>
 </robot>
